File: PCB_updi_unbricker.kicad_pcb (KiCad board)
At the start: 2 copper layers, 72 x 47.5 mm, 70 parts, among them J1 USB_C_Receptacle_USB2.0_16P, J2 Target, J3 TTL Serial, J4 RTS / DTR, J5 UPDI_TINY, J6 UPDI_DxEx, J7 UPDI_FW, Q1 BSS138, Q2 BSS84, Q3 BSS138, Q4 SSM3J332R, Q5 BSS84, Q6 BSS138, Q7 BSS84, Q8 BSS138, SW1 HV, SW2 VDD, SW3 Power, SW4 START, U1 CH340K, U2 LM1117GS-3.3, U3 MC34063AD, U4 ATtiny402-SS

Commit message: Update for Rev. 2 (PCBA)
Parts:
- removed C7: 0.1μ, Capacitor_THT:C_Disc_D3.0mm_W1.6mm_P2.50mm
- removed H1, H2, H3, H4: MountingHole, MountingHole:MountingHole_3.2mm_M3
- removed R6: 5.1, Resistor_THT:R_Axial_DIN0207_L6.3mm_D2.5mm_P2.54mm_Vertical
- removed R9: 200, Resistor_THT:R_Axial_DIN0207_L6.3mm_D2.5mm_P2.54mm_Vertical
- removed U3: MC34063AD, Library:DIP-8+SOIC-8
- added D12: 3.6V, Diode_THT:D_DO-35_SOD27_P2.54mm_Vertical_CathodeUp, F.Cu at (109.9, 49.5)
- added D13: 7.5V, Diode_THT:D_DO-41_SOD81_P2.54mm_Vertical_CathodeUp, F.Cu at (110.9, 60.3)
- added U5: MT3608, Package_TO_SOT_SMD:SOT-23-6, F.Cu at (104.6, 69.1)
- C1, C2: footprint Capacitor_SMD:C_1210_3225Metric -> Capacitor_SMD:C_0603_1608Metric
- C3: footprint Capacitor_THT:C_Disc_D3.0mm_W1.6mm_P2.50mm -> Capacitor_SMD:C_0603_1608Metric
- C4: value 100μ -> 22μ; footprint Capacitor_THT:CP_Radial_D5.0mm_P2.00mm -> Capacitor_SMD:C_0805_2012Metric
- C5: value 47μ -> 22μ; footprint Capacitor_THT:CP_Radial_D5.0mm_P2.00mm -> Capacitor_SMD:C_0805_2012Metric
- C6: value 220p -> 0.1μ; footprint Capacitor_THT:C_Disc_D3.0mm_W1.6mm_P2.50mm -> Capacitor_SMD:C_0603_1608Metric
- D1, D3, D4, D5, D6: value BAT43 -> BAT43WS; footprint Diode_THT:D_DO-35_SOD27_P2.54mm_Vertical_CathodeUp -> Diode_SMD:D_SOD-323
- D10: value 3V -> BZT52C7V5; footprint Diode_THT:D_DO-34_SOD68_P2.54mm_Vertical_CathodeUp -> Diode_SMD:D_SOD-123
- D11: value 5.1V -> 5.6V; footprint Diode_THT:D_DO-34_SOD68_P2.54mm_Vertical_CathodeUp -> Diode_THT:D_DO-41_SOD81_P2.54mm_Vertical_CathodeUp
- D2: value 5.6V -> BZT52C5V6; footprint Diode_THT:D_DO-35_SOD27_P2.54mm_Vertical_CathodeUp -> Diode_SMD:D_SOD-123
- D7: value 3.6V -> BZT52C3V6; footprint Diode_THT:D_DO-34_SOD68_P2.54mm_Vertical_CathodeUp -> Diode_SMD:D_SOD-123
- D8: value LED_Dual_AKA -> NCD0805R1; footprint LED_THT:LED_D5.0mm-3 -> LED_SMD:LED_0805_2012Metric
- D9: value 7.5V -> KT-0805G; footprint Diode_THT:D_DO-34_SOD68_P7.62mm_Horizontal -> LED_SMD:LED_0805_2012Metric
- F1: value Polyfuse_Small -> 0.5 A
- L1: value 330μ -> 4.7μ; footprint Resistor_THT:R_Axial_DIN0309_L9.0mm_D3.2mm_P2.54mm_Vertical -> Inductor_SMD:L_1210_3225Metric
- Q4: value SSM3J332R -> AO3401A
- R1, R14, R16, R17, R18, R19, R4, R7, R8: footprint Resistor_THT:R_Axial_DIN0207_L6.3mm_D2.5mm_P2.54mm_Vertical -> Resistor_SMD:R_0603_1608Metric
- R10: value 56k 1% -> 390k 1%; footprint Resistor_THT:R_Axial_DIN0207_L6.3mm_D2.5mm_P2.54mm_Vertical -> Resistor_SMD:R_0603_1608Metric
- R11: value 39k 1% -> 75k 1%; footprint Resistor_THT:R_Axial_DIN0207_L6.3mm_D2.5mm_P2.54mm_Vertical -> Resistor_SMD:R_0603_1608Metric
- R12: value 2.7k 1% -> 4.7k 1%; footprint Resistor_THT:R_Axial_DIN0207_L6.3mm_D2.5mm_P2.54mm_Vertical -> Resistor_SMD:R_0603_1608Metric
- R13: value 200 -> 220; footprint Resistor_THT:R_Axial_DIN0207_L6.3mm_D2.5mm_P2.54mm_Vertical -> Resistor_SMD:R_0603_1608Metric
- R15: value 4.7k -> 470; footprint Resistor_THT:R_Axial_DIN0207_L6.3mm_D2.5mm_P2.54mm_Vertical -> Resistor_SMD:R_0603_1608Metric
- R20: footprint Resistor_THT:R_Axial_DIN0204_L3.6mm_D1.6mm_P1.90mm_Vertical -> Resistor_SMD:R_0603_1608Metric
- R5: value 4.7k -> 220; footprint Resistor_THT:R_Axial_DIN0207_L6.3mm_D2.5mm_P2.54mm_Vertical -> Resistor_SMD:R_0603_1608Metric
- U1: footprint Library:SSOP-10-1EP_3.9x4.9mm_P1mm_EP2.1x3.3mm_HandSolder -> Package_SO:SSOP-10-1EP_3.9x4.9mm_P1mm_EP2.1x3.3mm
- U4: footprint Library:DIP-8+SOIC-8 -> Package_SO:SOIC-8_3.9x4.9mm_P1.27mm
- moved D11 58.4 mm to (76.2, 45.5), turned to -90 degrees
- moved C6 34.5 mm to (96.5, 76.2), turned to 0 degrees
- moved D9 28.6 mm to (101.0, 47.0), turned to 90 degrees
- moved D10 25.4 mm to (108.0, 59.1), turned to 90 degrees
- moved R5 23.0 mm to (104.0, 62.2)
- moved R15 21.8 mm to (104.1, 58.4)
- moved TP3 21.0 mm to (108.0, 54.6)
- moved C4 20.0 mm to (103.8, 72.4), turned to 180 degrees
- moved TP2 19.3 mm to (104.1, 54.6)
- moved C5 18.1 mm to (107.0, 65.4), turned to 180 degrees
- moved J3 17.8 mm to (120.1, 71.1)
- moved J5 17.8 mm to (115.6, 58.4)
- moved J6 17.8 mm to (115.6, 71.1)
- moved SW4 17.8 mm to (114.9, 76.5)
- moved D6 16.9 mm to (109.9, 66.0), turned to -90 degrees
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Connections:
- net Net-(J5-Pin_3) renamed /UPDI_TINY
- C3 pad 1: GND -> Net-(U1-V3)
- C3 pad 2: Net-(U1-V3) -> GND
- C4 pad 1: Net-(SW1-C) -> +5V
- C6 pad 1: Net-(U3-TC) -> +5V
- D10 pad 2: Net-(D10-A) -> GND
- D11 pad 1: Net-(D10-A) -> +5V
- D7 pad 2: Net-(D7-A) -> Net-(D12-A)
- D8 pad 1: Net-(D7-A) -> GND
- D8 pad 2: GND -> Net-(D12-A)
- D9 pad 1: +7.5V -> GND
- D9 pad 2: GND -> Net-(D9-A)
- L1 pad 1: Net-(U3-Ipk) -> +5V
- R14 pad 2: Net-(D8-A2) -> Net-(D9-A)
- SW1 pad 1: unconnected-(SW1-A-Pad1) -> GND
- SW1 pad 2: +5V -> Net-(SW1-B)
- SW1 pad 3: Net-(SW1-C) -> +5V
Routing:
- net GND: track 297.7 -> 110.5 mm, vias 8 -> 16
- net +5V: track 121.6 -> 58.3 mm
- net Net-(SW1-C): track 61.3 -> 0.00 mm, vias 1 -> 0
- net Net-(D6-A): track 39.0 -> 6.39 mm
- net INPUT: track 48.9 -> 22.0 mm
- net VDD_TGT: track 64.7 -> 39.1 mm
- net Net-(U3-Ipk): track 22.8 -> 0.00 mm, vias 1 -> 0
- net HV_75: track 58.6 -> 36.4 mm, vias 0 -> 1
- net Net-(U5-FB): track 28.5 -> 6.87 mm
- net Net-(SW1-B): track 0.00 -> 20.9 mm, vias 0 -> 1
- net UPDI_TGT: track 117.8 -> 98.2 mm, vias 4 -> 3
- net RTS/DTR: track 87.0 -> 68.4 mm, vias 0 -> 1
- net /RxD (TTL): track 62.5 -> 45.9 mm
- net CTS: track 89.0 -> 72.9 mm, vias 0 -> 1
- net Net-(U3-DC): track 15.8 -> 0.00 mm
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- added copper zone on F.Cu, net +5V
Other:
- board size 72 x 47.5 mm -> 54 x 47.5 mm
- board text added: "Rev.2"

Commit message: Fix R12 valude
Parts:
- R12: value 4.7k 1% -> 3.3k 1%
Changed lines of the file:
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@@
 			)
 		)
-		(property "Value" "4.7k 1%"
+		(property "Value" "3.3k 1%"
 			(at 0 1.43 0)
 			(layer "F.Fab")
